File: Trivia_Device.kicad_sch (KiCad schematic)
At the start: 0 parts

Commit message: trying to upload new version of schematic
Parts:
- added J1: Conn_01x24_Socket, symbol Connector:Conn_01x24_Socket
- added J2, J3: Conn_01x20_Socket, symbol Connector:Conn_01x20_Socket
- added U1: ~, symbol Custom:Fanstel_BC40C
Connections:
- no-connect marks 0 -> 2
